File: PC104Gus/hw/PC104GUS.kicad_pcb (KiCad board)
At the start: 2 copper layers, 95.9 x 90.2 mm, 63 parts, among them J1 Conn_02x32_Odd_Even, J10 Conn_02x30_Row_Letter_First, J11 AudioJack3, J12 AudioJack3, J2 Conn_02x20_Odd_Even, J3 Conn_01x02_Pin, J4 IRQDMA_JP, J5 Conn_01x04_Pin, J6 UART_TX, J9 Conn_02x30_Row_Letter_First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

Commit message: Board routing complete
DRC run, Need to update Schematic with parts from JLCPCB
Parts:
- moved FOX1 126.7 mm to (147.3, 64.8)
- moved C4 11.5 mm to (176.5, 86.9)
- moved C5 8.01 mm to (166.6, 84.2), turned to 180 degrees
- moved I2S_DAC1 7.57 mm to (158.1, 106.8)
- moved C2 1.80 mm to (172.6, 110.1), turned to 180 degrees
- moved C3 1.07 mm to (172.2, 98.9), turned to 180 degrees
Routing:
- net RUN: track 0.00 -> 101.6 mm, vias 0 -> 4
- net ~{RIOR}: track 0.00 -> 88.5 mm, vias 0 -> 3
- net ~{RIOW}: track 0.00 -> 87.6 mm, vias 0 -> 3
- net GND: track 0.00 -> 79.9 mm, vias 0 -> 70
- net ~{RI/OCHRDY}: track 0.00 -> 77.9 mm, vias 0 -> 2
- net D0: track 0.00 -> 72.3 mm, vias 0 -> 2
- net UART_TX: track 0.00 -> 72.1 mm, vias 0 -> 2
- net D2: track 0.00 -> 71.9 mm, vias 0 -> 2
- net D3: track 0.00 -> 70.5 mm, vias 0 -> 2
- net ~{BUSOE}: track 0.00 -> 70.0 mm, vias 0 -> 4
- net D1: track 0.00 -> 69.9 mm, vias 0 -> 2
- net ADS: track 0.00 -> 66.6 mm, vias 0 -> 4
- net D5: track 0.00 -> 66.3 mm, vias 0 -> 2
- net IRQ2: track 0.00 -> 65.9 mm, vias 0 -> 1
- net D4: track 0.00 -> 63.1 mm, vias 0 -> 2
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- added copper zone on In2.Cu, net +3V3
- added copper zone on In1.Cu, net GND
Other:
- copper layers 2 -> 4
- board text added: "PC104GUS V1.00 2025 Paula Maddox Based on"
- board text added: "PC104GUS, based on PicoGUS v1.2 © 2023 Ian Scott aka polpo licensed under CERN-OHL-P v2 https://github.com/polpo/picogus https://polpo.org/picogus"
- board text removed: "Leaded Solder Nicole Express PickledDog rasz_pl root42 Studio8502 SuperIlu TechAmbrosia Todd Gill tom7 Tube Time vswitchzero yyzkevin Zago everyone on Mastodon and Vogons everyone who contributed hardware or $$$ and the Retro Pico Hardware Discord for various combinations of inspiration, ideas, code, and/or help"
- board text removed: "PC104GUS V1.00 2025 Paula Maddox aka TechPaula Based on"
- board text removed: "thanks to: 48kRAM Aaron Giles Adrian Black Chrissy Claude Schwarz deck/scoopex djh0ffman FireTwoOneNine foone FreddyV furan Graham Sanderson HeathenUK indigoparadox Jim Leonard Jonathan Campbell Konrad Beckmann"
- board text removed: "v1.2 © 2023 Ian Scott aka polpo licensed under CERN-OHL-P v2 https://github.com/polpo/picogus https://polpo.org/picogus"
