File: PC104_Transputer/PC104_Transputer/PC104_Transputer.kicad_pcb (KiCad board)
At the start: 4 copper layers, 95.9 x 90.2 mm, 55 parts, among them J1 Conn_02x32_Odd_Even, J10 Conn_02x30_Row_Letter_First, J2 Conn_02x20_Odd_Even, J3 Conn_02x08_Odd_Even, J4 IRQDMA_JP, J5 Conn_02x05_Odd_Even, J9 Conn_02x30_Row_Letter_First, U11 IMSC011, U2 74LS244_Split, U4 74HC245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

Commit message: Board assembled, work on CPLD code
I found a bunch of mistakes in the CPLD equations, it's still not quite right yet
Parts:
- C2: value 100nF -> 1uF 10V
Changed lines of the file:
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@@
 			)
 		)
-		(property "Value" "100nF"
+		(property "Value" "1uF 10V"
 			(at 0 1.68 90)
 			(layer "F.Fab")
@@
 			)
 		)
+		(model "/home/paula/Dropbox/KiCAD/LIB/3D/10 pin female idc.step"
+			(offset
+				(xyz 1.25 -5 11)
+			)
+			(scale
+				(xyz 1 1 1)
+			)
+			(rotate
+				(xyz -90 -0 -90)
+			)
+		)
